File: electronics/invitation.sch (KiCad schematic (older format))
At the start: 22 parts, among them P1 USB_OTG, U1 ATMEGA32U4-A, X1 16 MHz

Commit message: Commit 37: Electronics business card initial design
Parts:
- removed X1: 16 MHz, Crystals:Resonator_7.2x3mm, symbol CRYSTAL_SMD
- added C3, C5: 22pF, Capacitors_SMD:C_0805, symbol C
- added P10: Tassimo, assets:tassimoButton, symbol CONN_01X01
- added P11: Maker, assets:makerButton, symbol CONN_01X01
- added P2: James Miller, assets:JMLogoButton, symbol CONN_01X01
- added P3: CONN_02X03, assets:Programming_port, symbol CONN_02X03
- added P4: D&AD, assets:moodButton, symbol CONN_01X01
- added P5: Krispy Kreme, assets:krispyButton, symbol CONN_01X01
- added P6: Epic Mind Drive, assets:mindDriveButton, symbol CONN_01X01
- added P7: Hacky Xmas, assets:hackyButton, symbol CONN_01X01
- added P8: Pay@Pump, assets:beerButton, symbol CONN_01X01
- added P9: WIYWI, assets:WiywiButton, symbol CONN_01X01
- added Y1: Crystal_Small, Crystals:Crystal_HC49-SD_SMD, symbol Crystal_Small
- D1: footprint (none) -> LEDs:LED_0402
- D2: renamed from D5; footprint (none) -> LEDs:LED_0402
- D3: renamed from D4; footprint (none) -> LEDs:LED_0402
- renumbered D3 to D4, D2 to D5
Connections:
- net labels added: MISO, MOSI, RESET, SCLK, heroBtn, portfolio1Btn, portfolio2Btn, portfolio3Btn, portfolio4Btn, portfolio5Btn, portfolio6Btn, portfolio7Btn, portfolio8Btn
- wire segments 70 -> 117
- no-connect marks 23 -> 14
Other:
- note added: "Buttons"
- note added: "Interaction LEDS"
- note added: "Programmer"
- moved on the sheet: D1, D2, D3, R4, R7, R8

Commit message: Commit 38: Business card pre-production
Parts:
- C3, C5: footprint Capacitors_SMD:C_0805 -> Capacitors_SMD:C_0402
- P10: footprint assets:tassimoButton -> assets:tassimoGif
- P11: footprint assets:makerButton -> assets:makerGif
- P2: footprint assets:JMLogoButton -> assets:JMLogo
- P4: footprint assets:moodButton -> assets:moodTreeGif
- P5: footprint assets:krispyButton -> assets:krispyKreme
- P6: footprint assets:mindDriveButton -> assets:mindDrive-F.Paste
- P7: footprint assets:hackyButton -> assets:hackyXmas
- P8: footprint assets:beerButton -> assets:beerGif-F.Paste
- P9: footprint assets:WiywiButton -> assets:WIYWI
- Y1: footprint Crystals:Crystal_HC49-SD_SMD -> assets:crystal_FA238-TSX3225
Connections:
- net labels added: Data+, Data-

Commit message: Commit 39: Business Card V1 Completed
Parts:
- D1: value Power LED -> Power LED (green)
- D2: value Interaction LED -> Interaction LED (green)
- D3: value Node LED -> Node LED (green)
- D4: value TX LED -> TX LED (orange)
- D5: value RX LED -> RX LED (orange)
- F1: value 500mA -> PPTC Fuse 500mA
- P1: value USB_OTG -> USB Micro B
- Y1: value Crystal_Small -> 16 FA-238 Mhz
Changed lines of the file:
@@
 P 1100 6400
 F 0 "P1" H 1425 6275 50  0000 C CNN
-F 1 "USB_OTG" H 1100 6600 50  0000 C CNN
+F 1 "USB Micro B" H 1100 6600 50  0000 C CNN
 F 2 "Connect:USB_Micro-B" V 1050 6300 50  0001 C CNN
 F 3 "" V 1050 6300 50  0000 C CNN
@@
 P 5250 2500
 F 0 "D4" H 5250 2600 50  0000 C CNN
-F 1 "TX LED" H 5250 2400 50  0000 C CNN
+F 1 "TX LED (orange)" H 5250 2400 50  0000 C CNN
 F 2 "LEDs:LED_0402" H 5250 2500 50  0001 C CNN
 F 3 "" H 5250 2500 50  0000 C CNN
@@
 P 5250 2000
 F 0 "D5" H 5250 2100 50  0000 C CNN
-F 1 "RX LED" H 5250 1900 50  0000 C CNN
+F 1 "RX LED (orange)" H 5250 1900 50  0000 C CNN
 F 2 "LEDs:LED_0402" H 5250 2000 50  0001 C CNN
 F 3 "" H 5250 2000 50  0000 C CNN
@@
 P 3800 6200
 F 0 "F1" H 3760 6260 50  0000 L CNN
-F 1 "500mA" H 3680 6140 50  0000 L CNN
+F 1 "PPTC Fuse 500mA" H 3680 6140 50  0000 L CNN
 F 2 "Fuse_Holders_and_Fuses:Fuse_SMD1206_Reflow" H 3800 6200 50  0001 C CNN
 F 3 "" H 3800 6200 50  0000 C CNN
@@
 P 9850 2200
 F 0 "D1" H 9850 2300 50  0000 C CNN
-F 1 "Power LED" H 9850 2100 50  0000 C CNN
+F 1 "Power LED (green)" H 9850 2100 50  0000 C CNN
 F 2 "LEDs:LED_0402" H 9850 2200 50  0001 C CNN
 F 3 "" H 9850 2200 50  0000 C CNN
@@
 P 9850 1750
 F 0 "D3" H 9850 1850 50  0000 C CNN
-F 1 "Node LED" H 9850 1650 50  0000 C CNN
+F 1 "Node LED (green)" H 9850 1650 50  0000 C CNN
 F 2 "LEDs:LED_0402" H 9850 1750 50  0001 C CNN
 F 3 "" H 9850 1750 50  0000 C CNN
@@
 P 9850 1400
 F 0 "D2" H 9850 1500 50  0000 C CNN
-F 1 "Interaction LED" H 9850 1300 50  0000 C CNN
+F 1 "Interaction LED (green)" H 9850 1300 50  0000 C CNN
 F 2 "LEDs:LED_0402" H 9850 1400 50  0001 C CNN
 F 3 "" H 9850 1400 50  0000 C CNN
@@
 P 1750 1900
 F 0 "Y1" H 1750 2000 50  0000 C CNN
-F 1 "Crystal_Small" H 1750 1800 50  0000 C CNN
+F 1 "16 FA-238 Mhz" H 1750 1800 50  0000 C CNN
 F 2 "assets:crystal_FA238-TSX3225" H 1750 1900 50  0001 C CNN
 F 3 "" H 1750 1900 50  0000 C CNN
