File: electronics/invitation.sch (KiCad schematic (older format))
At the start: 34 parts, among them P1 USB Micro B, P10 Tassimo, P11 Maker, P2 James Miller, P3 CONN_02X03, P4 D&AD, P5 Krispy Kreme, P6 Epic Mind Drive, P7 Hacky Xmas, P8 Pay@Pump, P9 WIYWI, U1 ATMEGA32U4-A, Y1 16 FA-238 Mhz

Commit message: Electronics
Parts:
- removed C1: 1uF, Capacitors_Tantalum_SMD:CP_Tantalum_Case-R_EIA-2012-12_Reflow, symbol CP1
- removed P10: Tassimo, assets:tassimoGif, symbol CONN_01X01
- removed P11: Maker, assets:makerGif, symbol CONN_01X01
- removed P3: CONN_02X03, assets:Programming_port, symbol CONN_02X03
- removed P6: Epic Mind Drive, assets:mindDrive-F.Paste, symbol CONN_01X01
- removed P7: Hacky Xmas, assets:hackyXmas, symbol CONN_01X01
- removed P8: Pay@Pump, assets:beerGif-F.Paste, symbol CONN_01X01
- removed P9: WIYWI, assets:WIYWI, symbol CONN_01X01
- added D6: TX LED (orange), LEDs:LED_0402, symbol LED
- added D7: RX LED (orange), LEDs:LED_0402, symbol LED
- added P3: Bottom Connections 1, Connectors_Samtec:SL-103-X-XX_1x03, symbol CONN_01X03
- added P6: Right Connectors, newAssets:SL-105-X-XX_1x05, symbol CONN_01X05
- added P7: Left Connectors, newAssets:SL-105-X-XX_1x05, symbol CONN_01X05
- added P8: Bottom Connections 2, Connectors_Samtec:SL-103-X-XX_1x03, symbol CONN_01X03
- added R10, R9: 330, Resistors_SMD:R_0402, symbol R
- D2: value Interaction LED (green) -> Website CTA (green)
- D3: value Node LED (green) -> Interaction LED (green)
- D4: value TX LED (orange) -> Phone LED (green)
- D5: value RX LED (orange) -> Email LED (green)
- P2: value James Miller -> Home button; footprint assets:JMLogo -> newAssets:JMDesign
- P4: value D&AD -> Left Arrow; footprint assets:moodTreeGif -> newAssets:leftArrow
- P5: value Krispy Kreme -> Right Arrow; footprint assets:krispyKreme -> newAssets:rightArrow
- R1, R2, R3, R4, R5, R6, R7, R8: footprint Resistors_SMD:R_0201 -> Resistors_SMD:R_0402
Connections:
- net labels added: A0, A1, A2, D0, D1, D2, D3, D4, RXLED, TXLED, XTal1, XTal2, emailLED, homeBtn, leftArrow, phoneLED, rightArrow
- net labels removed: heroBtn, portfolio1Btn, portfolio2Btn, portfolio3Btn, portfolio4Btn, portfolio5Btn, portfolio6Btn, portfolio7Btn, portfolio8Btn
- wire segments 117 -> 131
- no-connect marks 14 -> 7
Other:
- note added: "Crystal"
- note added: "Custom Pins"
- note added: "RX & TX LEDS"
- moved on the sheet: C3, C5, D1, D2, D3, D4, D5, F1, P2, P4, P5, R4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

Commit message: Business card updates
Parts:
- removed P7: Left Connectors, newAssets:SL-105-X-XX_1x05, symbol CONN_01X05
- removed P8: Bottom Connections 2, Connectors_Samtec:SL-103-X-XX_1x03, symbol CONN_01X03
- added P7: CONN_01X04, newAssets:SL-104-X-XX_1x04, symbol CONN_01X04
- added P8: CONN_01X01, newAssets:SL-101-X-XX_1x01, symbol CONN_01X01
- added P9: CONN_01X02, newAssets:SL-102-X-XX_1x02, symbol CONN_01X02
- C1: renamed from C5; footprint Capacitors_SMD:C_0201 -> Capacitors_SMD:C_0805
- C2: renamed from C3; footprint Capacitors_SMD:C_0201 -> Capacitors_SMD:C_0805
- C3: renamed from C4; footprint Capacitors_SMD:C_0201 -> Capacitors_SMD:C_0805
- D1, D2, D3: footprint LEDs:LED_0402 -> LEDs:LED_0805
- D4: renamed from D5; footprint LEDs:LED_0402 -> LEDs:LED_0805
- D5: renamed from D4; footprint LEDs:LED_0402 -> LEDs:LED_0805
- D6: renamed from D7; footprint LEDs:LED_0402 -> LEDs:LED_0805
- D7: renamed from D6; footprint LEDs:LED_0402 -> LEDs:LED_0805
- P3: footprint Connectors_Samtec:SL-103-X-XX_1x03 -> newAssets:SL-103-X-XX_1x03
- R1: renamed from R4; footprint Resistors_SMD:R_0402 -> Resistors_SMD:R_0805
- R10: renamed from R3; footprint Resistors_SMD:R_0402 -> Resistors_SMD:R_0805
- R2: renamed from R7; footprint Resistors_SMD:R_0402 -> Resistors_SMD:R_0805
- R3: renamed from R8; footprint Resistors_SMD:R_0402 -> Resistors_SMD:R_0805
- R4: renamed from R10; footprint Resistors_SMD:R_0402 -> Resistors_SMD:R_0805
- R5: renamed from R9; footprint Resistors_SMD:R_0402 -> Resistors_SMD:R_0805
- R6: renamed from R5; footprint Resistors_SMD:R_0402 -> Resistors_SMD:R_0805
- R7: renamed from R6; footprint Resistors_SMD:R_0402 -> Resistors_SMD:R_0805
- R8: renamed from R1; footprint Resistors_SMD:R_0402 -> Resistors_SMD:R_0805
- R9: renamed from R2; footprint Resistors_SMD:R_0402 -> Resistors_SMD:R_0805
- renumbered C2 to C0, C6 to C4, C7 to C5
