File: electronics/_autosave-invitation.kicad_pcb (KiCad board)
At the start: 2 copper layers, 86 x 57 mm, 62 parts, among them P1 USB Micro B, P10 Tassimo, P11 Maker, P2 James Miller, P3 CONN_02X03, P4 D&AD, P5 Krispy Kreme, P6 Epic Mind Drive, P7 Hacky Xmas, P8 Pay@Pump, P9 WIYWI, U1 ATMEGA32U4-A, Y1 16 FA-238 Mhz

Commit message: Commit 51: Re-adjusted Gerber files for production (silk screen layers too small + logo and maker project gifs needed resizing)
Parts:
- added P2: James Miller, assets:JMLogo, F.Cu at (161.8, 99.8)

Commit message: Commit 52: Final adjustment for PCB, now in production!!
Parts:
- added REF**: ESP-07v2, ESP8266:ESP-07v2, F.Cu at (105.4, 54.4)
Changed lines of the file:
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@@
     (links 86)
     (no_connects 1)
-    (area 119.169999 71.123999 205.320001 128.274001)
+    (area 114.707999 56.990001 218.162 130.910001)
     (thickness 1.6)
     (drawings 28)
     (tracks 794)
     (zones 0)
-    (modules 63)
+    (modules 64)
     (nets 45)
   )
@@
       (xy 4.124149 -1.152664) (xy 4.27489 -1.206397) (xy 4.282611 -1.2065) (xy 4.425696 -1.155825)) (layer F.Cu) (width 0.01))
   )
+  (module ESP8266:ESP-07v2 (layer F.Cu)
+    (at 105.41 54.356)
+    (descr "Module, ESP-8266, ESP-07v2, 16 pad, SMD")
+    (tags "Module ESP-8266 ESP8266")
+    (fp_text reference REF** (at -3.5 -1.5) (layer F.SilkS)
+      (effects (font (size 1 1) (thickness 0.15)))
+    )
+    (fp_text value ESP-07v2 (at 7.25 2.25) (layer F.Fab)
+      (effects (font (size 1 1) (thickness 0.15)))
+    )
+    (fp_line (start -2.25 -0.5) (end -2.25 -6.65) (layer F.CrtYd) (width 0.05))
+    (fp_line (start -2.25 -6.65) (end 16.25 -6.65) (layer F.CrtYd) (width 0.05))
+    (fp_line (start 16.25 -6.65) (end 16.25 16) (layer F.CrtYd) (width 0.05))
+    (fp_line (start 16.25 16) (end -2.25 16) (layer F.CrtYd) (width 0.05))
+    (fp_line (start -2.25 16) (end -2.25 -0.5) (layer F.CrtYd) (width 0.05))
+    (fp_line (start -1 -6.4) (end 15 -6.4) (layer F.SilkS) (width 0.1524))
+    (fp_line (start 15 -6.4) (end 15 -1) (layer F.SilkS) (width 0.1524))
+    (fp_line (start -1 -6.4) (end -1 -1) (layer F.SilkS) (width 0.1524))
+    (fp_line (start -1 14.8) (end -1 15.6) (layer F.SilkS) (width 0.1524))
+    (fp_line (start -1 15.6) (end 15 15.6) (layer F.SilkS) (width 0.1524))
+    (fp_line (start 15 15.6) (end 15 14.8) (layer F.SilkS) (width 0.1524))
+    (fp_line (start 15 -6.4) (end -1 -2.6) (layer F.SilkS) (width 0.1524))
+    (fp_line (start -1 -6.4) (end 15 -2.6) (layer F.SilkS) (width 0.1524))
+    (fp_text user "No Copper" (at 6.892 -5.4) (layer F.SilkS)
+      (effects (font (size 1 1) (thickness 0.15)))
+    )
+    (fp_line (start -1.008 -2.6) (end 14.992 -2.6) (layer F.SilkS) (width 0.1524))
+    (fp_line (start 15 -6.4) (end 15 15.6) (layer F.Fab) (width 0.05))
+    (fp_line (start 15 15.6) (end -1 15.6) (layer F.Fab) (width 0.05))
+    (fp_line (start -1.008 15.6) (end -1.008 -6.4) (layer F.Fab) (width 0.05))
+    (fp_line (start -1 -6.4) (end 15 -6.4) (layer F.Fab) (width 0.05))
+    (pad 1 thru_hole rect (at 0 0) (size 2.5 1.1) (drill 0.65 (offset -0.7 0)) (layers *.Cu *.Mask F.SilkS))
+    (pad 2 thru_hole oval (at 0 2) (size 2.5 1.1) (drill 0.65 (offset -0.7 0)) (layers *.Cu *.Mask F.SilkS))
+    (pad 3 thru_hole oval (at 0 4) (size 2.5 1.1) (drill 0.65 (offset -0.7 0)) (layers *.Cu *.Mask F.SilkS))
+    (pad 4 thru_hole oval (at 0 6) (size 2.5 1.1) (drill 0.65 (offset -0.7 0)) (layers *.Cu *.Mask F.SilkS))
+    (pad 5 thru_hole oval (at 0 8) (size 2.5 1.1) (drill 0.65 (offset -0.7 0)) (layers *.Cu *.Mask F.SilkS))
+    (pad 6 thru_hole oval (at 0 10) (size 2.5 1.1) (drill 0.65 (offset -0.7 0)) (layers *.Cu *.Mask F.SilkS))
+    (pad 7 thru_hole oval (at 0 12) (size 2.5 1.1) (drill 0.65 (offset -0.7 0)) (layers *.Cu *.Mask F.SilkS))
+    (pad 8 thru_hole oval (at 0 14) (size 2.5 1.1) (drill 0.65 (offset -0.7 0)) (layers *.Cu *.Mask F.SilkS))
+    (pad 9 thru_hole oval (at 14 14) (size 2.5 1.1) (drill 0.65 (offset 0.7 0)) (layers *.Cu *.Mask F.SilkS))
+    (pad 10 thru_hole oval (at 14 12) (size 2.5 1.1) (drill 0.65 (offset 0.6 0)) (layers *.Cu *.Mask F.SilkS))
+    (pad 11 thru_hole oval (at 14 10) (size 2.5 1.1) (drill 0.65 (offset 0.7 0)) (layers *.Cu *.Mask F.SilkS))
+    (pad 12 thru_hole oval (at 14 8) (size 2.5 1.1) (drill 0.65 (offset 0.7 0)) (layers *.Cu *.Mask F.SilkS))
+    (pad 13 thru_hole oval (at 14 6) (size 2.5 1.1) (drill 0.65 (offset 0.7 0)) (layers *.Cu *.Mask F.SilkS))
+    (pad 14 thru_hole oval (at 14 4) (size 2.5 1.1) (drill 0.65 (offset 0.7 0)) (layers *.Cu *.Mask F.SilkS))
+    (pad 15 thru_hole oval (at 14 2) (size 2.5 1.1) (drill 0.65 (offset 0.7 0)) (layers *.Cu *.Mask F.SilkS))
+    (pad 16 thru_hole oval (at 14 0) (size 2.5 1.1) (drill 0.65 (offset 0.7 0)) (layers *.Cu *.Mask F.SilkS))
+    (model ${ESPLIB}/ESP8266.3dshapes/ESP-07v2.wrl
+      (at (xyz 0 0 0))
+      (scale (xyz 0.3937 0.3937 0.3937))
+      (rotate (xyz 0 0 0))
+    )
+  )
   (dimension 57.15 (width 0.3) (layer Dwgs.User)
